File: hardware/uSafe.kicad_sch (KiCad schematic)
At the start: 1 part

Commit message: set up hardware
Parts:
- added C1, C2: 4.7uF, symbol Device:C
- added C3: 100uF, symbol Device:C
- added C4: 1nF, symbol Device:C
- added J1, J2: Conn_01x02_Socket, symbol Connector:Conn_01x02_Socket
- added L1: L, symbol Device:L
- added PS1: ITX4824SA-R, Converter_DCDC:Converter_DCDC_XP_POWER-ITxxxxxS_THT, symbol Converter_DCDC:ITX4824SA-R
- added Q1: BUZ11, Package_TO_SOT_THT:TO-220-3_Vertical, symbol Transistor_FET:BUZ11
Connections:
- net at A1.13 (GND), A1.18 (GND), A1.23 (GND)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: now also C3.2, C4.2, PS1.7 (-Vout)
- net at A1.36 (3V3): now also C3.1, PS1.6 (+Vout)
- new net: C1.1, J1.2 (Pin_2), J2.1 (Pin_1), L1.1
- new net: C2.1, L1.2, PS1.2 (+Vin)
- new net: C1.2, C2.2, C4.1, J1.1 (Pin_1), PS1.1 (-Vin), Q1.3 (S)
- new net: J2.2 (Pin_2), Q1.2 (D)
Other:
- moved on the sheet: A1

Commit message: started fleshing out hardware
Parts:
- added J3: Conn_01x08_Pin, symbol Connector:Conn_01x08_Pin
- added R1: R, Resistor_THT:R_Axial_DIN0207_L6.3mm_D2.5mm_P10.16mm_Horizontal, symbol Device:R
- A1: footprint Module:RaspberryPi_Pico_W_SMD_HandSolder -> Module:RaspberryPi_Pico_Common_THT
- C1, C2, C3, C4: footprint (none) -> Capacitor_THT:CP_Radial_Tantal_D5.0mm_P5.00mm
Connections:
- net at C3.1, PS1.6 (+Vout): now also A1.39 (VSYS); no longer A1.36 (3V3)
- net at A1.21 (GPIO16): now also J3.8 (Pin_8)
- net at A1.22 (GPIO17): now also J3.7 (Pin_7)
- net at A1.24 (GPIO18): now also J3.6 (Pin_6)
- net at A1.25 (GPIO19): now also J3.5 (Pin_5)
- net at A1.26 (GPIO20): now also J3.4 (Pin_4)
- net at A1.27 (GPIO21): now also J3.3 (Pin_3)
- net at A1.29 (GPIO22): now also J3.2 (Pin_2)
- net at A1.31 (GPIO26_ADC0): now also J3.1 (Pin_1)
- net at A1.37 (3V3_EN): now also R1.2
- net at A1.4 (GPIO2): now also Q1.1 (G)
- new net: A1.36 (3V3), R1.1

Commit message: added keypad connector
Parts:
- J1: footprint (none) -> Connector_JST:JST_EH_B2B-EH-A_1x02_P2.50mm_Vertical
- J3: footprint (none) -> Connector_JST:JST_EH_B8B-EH-A_1x08_P2.50mm_Vertical
Changed lines of the file:
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@@
 			)
 		)
-		(property "Footprint" ""
+		(property "Footprint" "Connector_JST:JST_EH_B8B-EH-A_1x08_P2.50mm_Vertical"
 			(at 217.17 105.41 0)
 			(effects
@@
 			)
 		)
-		(property "Footprint" ""
+		(property "Footprint" "Connector_JST:JST_EH_B2B-EH-A_1x02_P2.50mm_Vertical"
 			(at 26.67 66.04 0)
 			(effects
